File: kicad-files/rte.kicad_pcb (KiCad board)
At the start: 2 copper layers, 120 x 56 mm, 47 parts, among them J1 APU_LED_INPUT, J10 EXP_GPIO, J11 OC_BUFFER_OUTPUT, J12 APU_POWER_SUPPLY_INPUT, J13 APU_POWER_SUPPLY_OUTPUT, J14 RS232_OUT, J15 5V_POWER_SUPPLY, J17 USB_POWER_SUPPLY, J2 ORANGE_PI_ZERO_SERIAL_OUT, J3 ORANGE_PI_ZERO_GPIO2, J4 ORANGE_PI_ZERO_SERIAL_IN, J5 ORANGE_PI_ZERO_GPIO1, J6 USB_A1, J7 SPI_OUTPUT, J8 USB_A2, J9 I2C_BUS_OUTPUT, K1 HF3FA, Q1 NDS351AN, U1 MCP23017, U2 SN74LS06, U3 MAX3232, U4 SN74LS06

Commit message: Updated schematics to v1.0.0
Parts:
- added REF***: WEEE-Logo_4.2x6mm_SilkScreen, Symbols:WEEE-Logo_4.2x6mm_SilkScreen, F.Cu at (177.5, 96.7)
- C1, C2, C3, C4, C5, C6, C7: value 0.1uF -> 100nF; footprint Capacitors_SMD:C_1206_HandSoldering -> Capacitor_SMD:C_1206_3216Metric
- D2, D3: footprint Diodes_SMD:D_1206 -> Diode_SMD:D_1206_3216Metric
- F1: value FID1 -> Fiducial_1mm_Dia_2.54mm_Outer_CopperTop
- F2: value FID2 -> Fiducial_1mm_Dia_2.54mm_Outer_CopperTop
- F3: value FID3 -> Fiducial_1mm_Dia_2.54mm_Outer_CopperBottom; footprint Fiducials:Fiducial_1mm_Dia_2.54mm_Outer_CopperTop -> Fiducials:Fiducial_1mm_Dia_2.54mm_Outer_CopperBottom; moved to F.Cu
- F4: value FID4 -> Fiducial_1mm_Dia_2.54mm_Outer_CopperBottom; footprint Fiducials:Fiducial_1mm_Dia_2.54mm_Outer_CopperTop -> Fiducials:Fiducial_1mm_Dia_2.54mm_Outer_CopperBottom; moved to F.Cu
- G1: footprint Documents:3mdeb_logo -> footprints:3mdeb_logo
- J1: footprint Pin_Headers:Pin_Header_Straight_1x03_Pitch2.54mm -> Connector_PinHeader_2.54mm:PinHeader_1x03_P2.54mm_Vertical
- J10: value EXP_GPIO -> EXP_GPIO_OUTPUT; footprint Pin_Headers:Pin_Header_Straight_1x04_Pitch2.54mm -> Connector_PinHeader_2.54mm:PinHeader_1x04_P2.54mm_Vertical
- J11: footprint Pin_Headers:Pin_Header_Straight_1x12_Pitch2.54mm -> Connector_PinHeader_2.54mm:PinHeader_1x12_P2.54mm_Vertical
- J12, J13: footprint Connectors:Barrel_Jack_CUI_PJ-102AH -> Connector_BarrelJack:BarrelJack_CUI_PJ-102AH_Horizontal
- J14: footprint Connectors2:DB9MD -> Connect:DB9MD
- J15: footprint Pin_Headers:Pin_Header_Straight_1x02_Pitch2.54mm -> Connector_PinHeader_2.54mm:PinHeader_1x02_P2.54mm_Vertical
- J3: value ORANGE_PI_ZERO_GPIO2 -> ORANGE_PI_ZERO_CONN2; footprint Pin_Headers:Pin_Header_Straight_1x13_Pitch2.54mm -> Connector_PinSocket_2.54mm:PinSocket_1x13_P2.54mm_Vertical; moved to B.Cu
- J4: footprint Pin_Headers:Pin_Header_Straight_1x03_Pitch2.54mm -> Connector_PinSocket_2.54mm:PinSocket_1x03_P2.54mm_Vertical; moved to B.Cu
- J5: value ORANGE_PI_ZERO_GPIO1 -> ORANGE_PI_ZERO_CONN1; footprint Pin_Headers:Pin_Header_Straight_2x13_Pitch2.54mm -> Connector_PinSocket_2.54mm:PinSocket_2x13_P2.54mm_Vertical; moved to B.Cu
- J7: footprint Pin_Headers:Pin_Header_Straight_2x04_Pitch2.54mm -> Connector_PinHeader_2.54mm:PinHeader_2x04_P2.54mm_Vertical
- J9: footprint Pin_Headers:Pin_Header_Straight_1x04_Pitch2.54mm -> Connector_PinHeader_2.54mm:PinHeader_1x04_P2.54mm_Vertical
- R1, R2, R3: footprint Resistors_SMD:R_1206_HandSoldering -> Resistor_SMD:R_1206_3216Metric
- U1: footprint Housings_SOIC:SOIC-28W_7.5x17.9mm_Pitch1.27mm -> Package_SO:SOIC-28W_7.5x17.9mm_P1.27mm
- U2, U4: value SN74LS06 -> 74LS06; footprint Housings_SOIC:SOIC-14_3.9x8.7mm_Pitch1.27mm -> Package_SO:SOIC-14_3.9x8.7mm_P1.27mm
- U3: footprint SMD_Packages:SO-16-N -> Package_SO:SOIC-16_3.9x9.9mm_P1.27mm
- moved J14 5.62 mm to (180.1, 122.8)
- moved G1 3.84 mm to (174.1, 90.0)
- moved F1 2.69 mm to (118.3, 116.0)
- moved F2 2.17 mm to (198.2, 122.0)
- moved F4 1.54 mm to (130.0, 109.8)
- moved C6 0.96 mm to (167.6, 101.4)
- moved R3 0.50 mm to (184.0, 104.7)
- moved R1 0.41 mm to (114.1, 116.4)
- moved F3 0.13 mm to (198.3, 118.1)
- turned J5 to 90 degrees
- turned J3 to 90 degrees
- turned J4 to 270 degrees
- turned U3 to 0 degrees
Connections:
- J14 pad 1: Net-(J14-Pad1) -> (no net)
- J14 pad 4: Net-(J14-Pad4) -> (no net)
- J14 pad 6: Net-(J14-Pad6) -> (no net)
- J14 pad 9: Net-(J14-Pad9) -> (no net)
- J17 pad 2: Net-(J17-Pad2) -> (no net)
- J17 pad 3: Net-(J17-Pad3) -> (no net)
- J17 pad 4: Net-(J17-Pad4) -> (no net)
- J3 pad 1: Net-(J3-Pad1) -> (no net)
- J3 pad 2: Net-(J3-Pad2) -> (no net)
- J3 pad 3: Net-(J3-Pad3) -> (no net)
- J3 pad 4: Net-(J3-Pad4) -> (no net)
- J3 pad 5: Net-(J3-Pad5) -> (no net)
- J3 pad 6: Net-(J3-Pad6) -> (no net)
- J3 pad 7: Net-(J3-Pad7) -> (no net)
- J5 pad 8: Net-(J5-Pad8) -> (no net)
- J7 pad 1: Net-(J7-Pad1) -> (no net)
- J7 pad 7: Net-(J7-Pad7) -> (no net)
- J7 pad 8: Net-(J7-Pad8) -> (no net)
- K1 pad 4: Net-(K1-Pad4) -> (no net)
Routing:
- net +5V: track 207.9 -> 195.1 mm
- net USB_DP2: track 56.5 -> 44.4 mm, vias 0 -> 1
- net USB_DM3: track 63.6 -> 51.7 mm
- net USB_DP3: track 62.1 -> 51.7 mm, vias 0 -> 2
- net GND: track 6.19 -> 11.9 mm
- net UART2_RTS: track 106.5 -> 102.8 mm
- net Net-(D1-Pad2): track 32.7 -> 30.2 mm
- net RELAY_CTR: track 85.8 -> 84.0 mm
- net E_GPB1: track 19.2 -> 21.0 mm
- net E_GPB3: track 24.8 -> 26.6 mm
- net E_GPB2: track 24.2 -> 26.0 mm
- net Net-(C6-Pad1): track 6.25 -> 7.86 mm
- net E_GPB4: track 24.7 -> 26.3 mm
- net OC_OUT2: track 9.34 -> 10.6 mm
- net UART2_RX: track 83.5 -> 82.4 mm
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Other:
- board size 120 x 56 mm -> 120.1 x 56 mm
- board text added: "RTE board v1.0.0"
- board text added: "RoHS"
- board text removed: "RTE board v.0.5.3"
