File: kicad-files/rte.sch (KiCad schematic (older format))
At the start: 42 parts, among them J1 APU_LED_INPUT, J10 EXP_GPIO_OUTPUT, J11 OC_BUFFER_OUTPUT, J12 APU_POWER_SUPPLY_INPUT, J13 APU_POWER_SUPPLY_OUTPUT, J14 RS232_OUT, J15 5V_POWER_SUPPLY, J17 USB_POWER_SUPPLY, J2 ORANGE_PI_ZERO_SERIAL_OUT, J3 ORANGE_PI_ZERO_CONN2, J4 ORANGE_PI_ZERO_SERIAL_IN, J5 ORANGE_PI_ZERO_CONN1, J6 USB_A1, J7 SPI_OUTPUT, J8 USB_A2, J9 I2C_BUS_OUTPUT, K1 HF3FA, Q1 NDS351AN, U1 MCP23017, U2 SN74LS06, U3 MAX3232, U4 SN74LS06

Commit message: Updated schematics to v1.0.0
Parts:
- removed C1, C2, C3, C5, C6, C7: 0.1uF, Capacitors_SMD:C_1206_HandSoldering, symbol C
- removed U2, U4: SN74LS06, Housings_SOIC:SOIC-14_3.9x8.7mm_Pitch1.27mm, symbol SN74LS06
- added C1, C2, C4, C5, C6, C7: 100nF, Capacitor_SMD:C_1206_3216Metric, symbol rte:C
- added U2, U4: 74LS06, Package_SO:SOIC-14_3.9x8.7mm_P1.27mm, symbol 3mdeb:74LS06
- C3: renamed from C4; value 0.1uF -> 100nF; footprint Capacitors_SMD:C_1206_HandSoldering -> Capacitor_SMD:C_1206_3216Metric; symbol C -> rte:C
- D1: symbol D_ALT -> rte:D_ALT
- D2, D3: footprint Diodes_SMD:D_1206 -> Diode_SMD:D_1206_3216Metric; symbol LED_ALT -> rte:LED_ALT
- J1: footprint Pin_Headers:Pin_Header_Straight_1x03_Pitch2.54mm -> Connector_PinHeader_2.54mm:PinHeader_1x03_P2.54mm_Vertical; symbol Conn_01x03 -> rte:Conn_01x03
- J10, J9: footprint Pin_Headers:Pin_Header_Straight_1x04_Pitch2.54mm -> Connector_PinHeader_2.54mm:PinHeader_1x04_P2.54mm_Vertical; symbol Conn_01x04 -> rte:Conn_01x04
- J11: footprint Pin_Headers:Pin_Header_Straight_1x12_Pitch2.54mm -> Connector_PinHeader_2.54mm:PinHeader_1x12_P2.54mm_Vertical; symbol Conn_01x12 -> rte:Conn_01x12
- J12, J13: footprint Connectors:Barrel_Jack_CUI_PJ-102AH -> Connector_BarrelJack:BarrelJack_CUI_PJ-102AH_Horizontal; symbol Barrel_Jack -> rte:Barrel_Jack
- J14: footprint Connectors:DB9FD -> Connect:DB9MD; symbol DB9_Male_MountingHoles -> rte:DB9_Male_MountingHoles
- J15: footprint Pin_Headers:Pin_Header_Straight_1x02_Pitch2.54mm -> Connector_PinHeader_2.54mm:PinHeader_1x02_P2.54mm_Vertical; symbol Conn_01x02 -> rte:Conn_01x02
- J17: symbol USB_OTG-RESCUE-remote_development_board -> rte:USB_OTG-RESCUE-remote_development_board
- J2: symbol Conn_01x03 -> rte:Conn_01x03
- J3: footprint Pin_Headers:Pin_Header_Straight_1x13_Pitch2.54mm -> Connector_PinSocket_2.54mm:PinSocket_1x13_P2.54mm_Vertical; symbol Conn_01x13 -> rte:Conn_01x13
- J4: footprint Pin_Headers:Pin_Header_Straight_1x03_Pitch2.54mm -> Connector_PinSocket_2.54mm:PinSocket_1x03_P2.54mm_Vertical; symbol Conn_01x03 -> rte:Conn_01x03
- J5: footprint Pin_Headers:Pin_Header_Straight_2x13_Pitch2.54mm -> Connector_PinSocket_2.54mm:PinSocket_2x13_P2.54mm_Vertical; symbol Conn_02x13_Odd_Even -> rte:Conn_02x13_Odd_Even
- J6, J8: symbol USB_A-RESCUE-remote_development_board -> rte:USB_A-RESCUE-remote_development_board
- J7: footprint Pin_Headers:Pin_Header_Straight_2x04_Pitch2.54mm -> Connector_PinHeader_2.54mm:PinHeader_2x04_P2.54mm_Vertical; symbol Conn_02x04_Odd_Even -> rte:Conn_02x04_Odd_Even
- K1: symbol HF3-51-RESCUE-remote_development_board -> rte:HF3-51-RESCUE-remote_development_board
- MK1, MK2, MK3, MK4, MK5, MK6, MK7: symbol Mounting_Hole -> rte:Mounting_Hole
- Q1: symbol Q_NMOS_DGS-RESCUE-remote_development_board -> rte:Q_NMOS_DGS-RESCUE-remote_development_board
- R1, R2, R3: footprint Resistors_SMD:R_1206_HandSoldering -> Resistor_SMD:R_1206_3216Metric; symbol R -> rte:R
- U1: footprint Housings_SOIC:SOIC-28W_7.5x17.9mm_Pitch1.27mm -> Package_SO:SOIC-28W_7.5x17.9mm_P1.27mm; symbol MCP23017 -> rte:MCP23017
- U3: footprint SMD_Packages:SO-16-N -> Package_SO:SOIC-16_3.9x9.9mm_P1.27mm; symbol MAX3232 -> rte:MAX3232
Connections:
- wire segments 220 -> 245
Other:
- note removed: "0.5.3"
- note removed: "01.02.2018"
- note removed: "Remote Testing Environment"
- note removed: "Remote Testing Environment schematic \nv.0.5.3"
